File: rabbit LEDs.kicad_sch (KiCad schematic)
At the start: 24 parts

Commit message: Add BoM and complete board
Parts:
- R13, R14, R15, R16, R17, R18, R19, R20, R21, R22, R23, R24: value 500 -> 82
Changed lines of the file:
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@@
       (effects (font (size 1.27 1.27)) (justify left))
     )
-    (property "Value" "500" (id 1) (at 77.47 74.9299 0)
+    (property "Value" "82" (id 1) (at 77.47 74.9299 0)
       (effects (font (size 1.27 1.27)) (justify left))
     )
@@
       (effects (font (size 1.27 1.27)) (justify left))
     )
-    (property "Value" "500" (id 1) (at 181.61 74.9299 0)
+    (property "Value" "82" (id 1) (at 181.61 74.9299 0)
       (effects (font (size 1.27 1.27)) (justify left))
     )
@@
       (effects (font (size 1.27 1.27)) (justify left))
     )
-    (property "Value" "500" (id 1) (at 63.5 74.9299 0)
+    (property "Value" "82" (id 1) (at 63.5 74.9299 0)
       (effects (font (size 1.27 1.27)) (justify left))
     )
@@
       (effects (font (size 1.27 1.27)) (justify left))
     )
-    (property "Value" "500" (id 1) (at 102.87 74.9299 0)
+    (property "Value" "82" (id 1) (at 102.87 74.9299 0)
       (effects (font (size 1.27 1.27)) (justify left))
     )
@@
       (effects (font (size 1.27 1.27)) (justify left))
     )
-    (property "Value" "500" (id 1) (at 142.24 74.9299 0)
+    (property "Value" "82" (id 1) (at 142.24 74.9299 0)
       (effects (font (size 1.27 1.27)) (justify left))
     )
@@
       (effects (font (size 1.27 1.27)) (justify left))
     )
-    (property "Value" "500" (id 1) (at 208.28 74.9299 0)
+    (property "Value" "82" (id 1) (at 208.28 74.9299 0)
       (effects (font (size 1.27 1.27)) (justify left))
     )
@@
       (effects (font (size 1.27 1.27)) (justify left))
     )
-    (property "Value" "500" (id 1) (at 195.58 74.9299 0)
+    (property "Value" "82" (id 1) (at 195.58 74.9299 0)
       (effects (font (size 1.27 1.27)) (justify left))
     )
@@
       (effects (font (size 1.27 1.27)) (justify left))
     )
-    (property "Value" "500" (id 1) (at 90.17 74.9299 0)
+    (property "Value" "82" (id 1) (at 90.17 74.9299 0)
       (effects (font (size 1.27 1.27)) (justify left))
     )
@@
       (effects (font (size 1.27 1.27)) (justify left))
     )
-    (property "Value" "500" (id 1) (at 156.21 74.9299 0)
+    (property "Value" "82" (id 1) (at 156.21 74.9299 0)
       (effects (font (size 1.27 1.27)) (justify left))
     )
@@
       (effects (font (size 1.27 1.27)) (justify left))
     )
-    (property "Value" "500" (id 1) (at 129.54 74.9299 0)
+    (property "Value" "82" (id 1) (at 129.54 74.9299 0)
       (effects (font (size 1.27 1.27)) (justify left))
     )
@@
       (effects (font (size 1.27 1.27)) (justify left))
     )
-    (property "Value" "500" (id 1) (at 116.84 74.9299 0)
+    (property "Value" "82" (id 1) (at 116.84 74.9299 0)
       (effects (font (size 1.27 1.27)) (justify left))
     )
@@
       (effects (font (size 1.27 1.27)) (justify left))
     )
-    (property "Value" "500" (id 1) (at 168.91 74.9299 0)
-      (effects (font (size 1.27 1.27)) (justify left))
-    )
+    (property "Value" "82" (id 1) (at 168.91 74.9299 0)
+      (effects (font (size 1.27 1.27)) (justify left))
+    )
